File: eagle/midi_to_cv.sch (EAGLE design)
At the start: 66 parts, among them IC1 4093N, Q3 2N3904, Q4 2N3904, Q5 2N3904, Q6 2SK30, U1 ATMEGA328P_PDIP

Commit message: arduino code compiles
Parts:
- C8: value 470pF -> 10n
- R10: value 1M5 -> 2M2
- R9: value 68k -> 100k
Changed lines of the file:
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@@
 <?xml version="1.0" encoding="utf-8"?>
 <!DOCTYPE eagle SYSTEM "eagle.dtd">
-<eagle version="7.6.0">
+<eagle version="7.1.0">
 <drawing>
 <settings>
@@
 <part name="R7" library="rcl" deviceset="R-US_" device="0204/7" value="1M"/>
 <part name="GND8" library="supply1" deviceset="GND" device=""/>
-<part name="R9" library="rcl" deviceset="R-US_" device="0204/7" value="68k"/>
-<part name="C8" library="rcl" deviceset="C-US" device="025-040X050" value="470pF"/>
+<part name="R9" library="rcl" deviceset="R-US_" device="0204/7" value="100k"/>
+<part name="C8" library="rcl" deviceset="C-US" device="025-040X050" value="10n"/>
 <part name="Q4" library="808_lt" deviceset="2N3904" device=""/>
-<part name="R10" library="rcl" deviceset="R-US_" device="0204/7" value="1M5"/>
+<part name="R10" library="rcl" deviceset="R-US_" device="0204/7" value="2M2"/>
 <part name="Q5" library="808_lt" deviceset="2N3904" device=""/>
 <part name="GND9" library="supply1" deviceset="GND" device=""/>
